File: gadget.kicad_pcb (KiCad board)
At the start: 2 copper layers, 69.4 x 71.2 mm, 50 parts, among them J1 Conn_01x04_Pin, J2 Conn_01x04_Pin, J3 Conn_01x04_Pin, J4 Conn_01x04_Pin, J5 Conn_01x04_Pin, U1 CH32V003JxMx

Commit message: jignesh
Other:
- board text added: "fallout 2026"
- board text added: "kermicidal.xyz"
